Commit message: add bed trolley

File: ranger_mini_v2_gazebo/xacro/rangerminibedtrolly.xacro (robot description, xacro)
@@ -1,4 +1,4 @@
 <?xml version="1.0"?>
-<robot name="ranger_mini_patient_chair"
+<robot name="rangerminibedtrolly"
     xmlns:xacro="http://ros.org/wiki/xacro">
     <!-- Material definitions -->
@@ -15,9 +15,12 @@
         <color rgba="0.7 0.7 0.7 1" />
     </material>
-    <material name="chair_black">
-        <color rgba="0.05 0.05 0.05 1" />
-    </material>
-    <material name="chair_metal">
-        <color rgba="0.8 0.8 0.8 1" />
+    <material name="bed_blue">
+        <color rgba="0.2 0.4 0.8 1" />
+    </material>
+    <material name="bed_white">
+        <color rgba="0.95 0.95 0.95 1" />
+    </material>
+    <material name="bed_metal">
+        <color rgba="0.6 0.6 0.6 1" />
     </material>
     <!-- Base link -->
@@ -41,4 +44,159 @@
         </collision>
     </link>
+    <!-- Support cylinder for bed -->
+    <link name="bed_support_link">
+        <inertial>
+            <origin xyz="0.0 0.0 0.0"/>
+            <mass value="5"/>
+            <inertia ixx="0.1" ixy="0.0" ixz="0.0" iyy="0.1" iyz="0.0" izz="0.1"/>
+        </inertial>
+        <visual>
+            <origin xyz="0 0 0" rpy="0 0 0" />
+            <geometry>
+                <cylinder radius="0.05" length="0.8"/>
+            </geometry>
+            <material name="bed_metal"/>
+        </visual>
+        <collision>
+            <origin xyz="0 0 0" rpy="0 0 0" />
+            <geometry>
+                <cylinder radius="0.05" length="0.8"/>
+            </geometry>
+        </collision>
+    </link>
+    <joint name="bed_support_joint" type="fixed">
+        <origin xyz="0.3 0 0.1" rpy="0 0 0" />
+        <parent link="base_link"/>
+        <child link="bed_support_link"/>
+    </joint>
+    <!-- Bed structure -->
+    <link name="bed_frame_link">
+        <inertial>
+            <origin xyz="0.0 0.0 0.0"/>
+            <mass value="15"/>
+            <inertia ixx="0.5" ixy="0.0" ixz="0.0" iyy="0.5" iyz="0.0" izz="0.5"/>
+        </inertial>
+        <visual>
+            <origin xyz="0 0 0" rpy="0 0 0" />
+            <geometry>
+                <box size="1.8 0.8 0.1"/>
+            </geometry>
+            <material name="bed_metal"/>
+        </visual>
+        <collision>
+            <origin xyz="0 0 0" rpy="0 0 0" />
+            <geometry>
+                <box size="1.8 0.8 0.1"/>
+            </geometry>
+        </collision>
+    </link>
+    <joint name="bed_frame_joint" type="fixed">
+        <origin xyz="0 0 0.45" rpy="0 0 0" />
+        <parent link="bed_support_link"/>
+        <child link="bed_frame_link"/>
+    </joint>
+    <!-- Bed mattress -->
+    <link name="bed_mattress_link">
+        <inertial>
+            <origin xyz="0.0 0.0 0.0"/>
+            <mass value="8"/>
+            <inertia ixx="0.3" ixy="0.0" ixz="0.0" iyy="0.3" iyz="0.0" izz="0.3"/>
+        </inertial>
+        <visual>
+            <origin xyz="0 0 0" rpy="0 0 0" />
+            <geometry>
+                <box size="1.7 0.7 0.08"/>
+            </geometry>
+            <material name="bed_blue"/>
+        </visual>
+        <collision>
+            <origin xyz="0 0 0" rpy="0 0 0" />
+            <geometry>
+                <box size="1.7 0.7 0.08"/>
+            </geometry>
+        </collision>
+    </link>
+    <joint name="bed_mattress_joint" type="fixed">
+        <origin xyz="0 0 0.09" rpy="0 0 0" />
+        <parent link="bed_frame_link"/>
+        <child link="bed_mattress_link"/>
+    </joint>
+    <!-- Bed headboard -->
+    <link name="bed_headboard_link">
+        <inertial>
+            <origin xyz="0.0 0.0 0.0"/>
+            <mass value="3"/>
+            <inertia ixx="0.1" ixy="0.0" ixz="0.0" iyy="0.1" iyz="0.0" izz="0.1"/>
+        </inertial>
+        <visual>
+            <origin xyz="0 0 0" rpy="0 0 0" />
+            <geometry>
+                <box size="0.05 0.8 0.4"/>
+            </geometry>
+            <material name="bed_white"/>
+        </visual>
+        <collision>
+            <origin xyz="0 0 0" rpy="0 0 0" />
+            <geometry>
+                <box size="0.05 0.8 0.4"/>
+            </geometry>
+        </collision>
+    </link>
+    <joint name="bed_headboard_joint" type="fixed">
+        <origin xyz="0.925 0 0.2" rpy="0 0 0" />
+        <parent link="bed_frame_link"/>
+        <child link="bed_headboard_link"/>
+    </joint>
+    <!-- Bed side rails -->
+    <link name="bed_rail_left_link">
+        <inertial>
+            <origin xyz="0.0 0.0 0.0"/>
+            <mass value="2"/>
+            <inertia ixx="0.05" ixy="0.0" ixz="0.0" iyy="0.05" iyz="0.0" izz="0.05"/>
+        </inertial>
+        <visual>
+            <origin xyz="0 0 0" rpy="0 0 0" />
+            <geometry>
+                <box size="1.8 0.03 0.3"/>
+            </geometry>
+            <material name="bed_metal"/>
+        </visual>
+        <collision>
+            <origin xyz="0 0 0" rpy="0 0 0" />
+            <geometry>
+                <box size="1.8 0.03 0.3"/>
+            </geometry>
+        </collision>
+    </link>
+    <joint name="bed_rail_left_joint" type="fixed">
+        <origin xyz="0 -0.415 0.15" rpy="0 0 0" />
+        <parent link="bed_frame_link"/>
+        <child link="bed_rail_left_link"/>
+    </joint>
+    <link name="bed_rail_right_link">
+        <inertial>
+            <origin xyz="0.0 0.0 0.0"/>
+            <mass value="2"/>
+            <inertia ixx="0.05" ixy="0.0" ixz="0.0" iyy="0.05" iyz="0.0" izz="0.05"/>
+        </inertial>
+        <visual>
+            <origin xyz="0 0 0" rpy="0 0 0" />
+            <geometry>
+                <box size="1.8 0.03 0.3"/>
+            </geometry>
+            <material name="bed_metal"/>
+        </visual>
+        <collision>
+            <origin xyz="0 0 0" rpy="0 0 0" />
+            <geometry>
+                <box size="1.8 0.03 0.3"/>
+            </geometry>
+        </collision>
+    </link>
+    <joint name="bed_rail_right_joint" type="fixed">
+        <origin xyz="0 0.415 0.15" rpy="0 0 0" />
+        <parent link="bed_frame_link"/>
+        <child link="bed_rail_right_link"/>
+    </joint>
    <link name="fl_steering_wheel_link">
         <inertial>
@@ -271,159 +429,4 @@
             <axis xyz="0 1 0" rpy="0 0 0" />
         </joint>
-    <!-- Chair Structure -->
-    <!-- Chair Seat -->
-    <link name="chair_seat">
-        <inertial>
-            <origin xyz="0.0 0.0 0.0"/>
-            <mass value="5"/>
-            <inertia ixx="0.2" ixy="0.0" ixz="0.0" iyy="0.2" iyz="0.0" izz="0.2"/>
-        </inertial>
-        <visual>
-            <origin xyz="0 0 0" rpy="0 0 0" />
-            <geometry>
-                <box size="0.4 0.35 0.05" />
-            </geometry>
-            <material name="chair_black" />
-        </visual>
-        <collision>
-            <origin xyz="0 0 0" rpy="0 0 0" />
-            <geometry>
-                <box size="0.4 0.35 0.05" />
-            </geometry>
-        </collision>
-    </link>
-    <!-- Chair Back -->
-    <link name="chair_back">
-        <inertial>
-            <origin xyz="0.0 0.0 0.0"/>
-            <mass value="3"/>
-            <inertia ixx="0.1" ixy="0.0" ixz="0.0" iyy="0.1" iyz="0.0" izz="0.1"/>
-        </inertial>
-        <visual>
-            <origin xyz="0 0 0" rpy="0 0 0" />
-            <geometry>
-                <box size="0.4 0.05 0.4" />
-            </geometry>
-            <material name="chair_black" />
-        </visual>
-        <collision>
-            <origin xyz="0 0 0" rpy="0 0 0" />
-            <geometry>
-                <box size="0.4 0.05 0.4" />
-            </geometry>
-        </collision>
-    </link>
-    <!-- Chair Legs -->
-    <link name="chair_leg1">
-        <inertial>
-            <origin xyz="0.0 0.0 0.0"/>
-            <mass value="1"/>
-            <inertia ixx="0.01" ixy="0.0" ixz="0.0" iyy="0.01" iyz="0.0" izz="0.01"/>
-        </inertial>
-        <visual>
-            <origin xyz="0 0 0" rpy="0 0 0" />
-            <geometry>
-                <cylinder length="0.3" radius="0.01" />
-            </geometry>
-            <material name="chair_metal" />
-        </visual>
-        <collision>
-            <origin xyz="0 0 0" rpy="0 0 0" />
-            <geometry>
-                <cylinder length="0.3" radius="0.01" />
-            </geometry>
-        </collision>
-    </link>
-    <link name="chair_leg2">
-        <inertial>
-            <origin xyz="0.0 0.0 0.0"/>
-            <mass value="1"/>
-            <inertia ixx="0.01" ixy="0.0" ixz="0.0" iyy="0.01" iyz="0.0" izz="0.01"/>
-        </inertial>
-        <visual>
-            <origin xyz="0 0 0" rpy="0 0 0" />
-            <geometry>
-                <cylinder length="0.3" radius="0.01" />
-            </geometry>
-            <material name="chair_metal" />
-        </visual>
-        <collision>
-            <origin xyz="0 0 0" rpy="0 0 0" />
-            <geometry>
-                <cylinder length="0.3" radius="0.01" />
-            </geometry>
-        </collision>
-    </link>
-    <link name="chair_leg3">
-        <inertial>
-            <origin xyz="0.0 0.0 0.0"/>
-            <mass value="1"/>
-            <inertia ixx="0.01" ixy="0.0" ixz="0.0" iyy="0.01" iyz="0.0" izz="0.01"/>
-        </inertial>
-        <visual>
-            <origin xyz="0 0 0" rpy="0 0 0" />
-            <geometry>
-                <cylinder length="0.3" radius="0.01" />
-            </geometry>
-            <material name="chair_metal" />
-        </visual>
-        <collision>
-            <origin xyz="0 0 0" rpy="0 0 0" />
-            <geometry>
-                <cylinder length="0.3" radius="0.01" />
-            </geometry>
-        </collision>
-    </link>
-    <link name="chair_leg4">
-        <inertial>
-            <origin xyz="0.0 0.0 0.0"/>
-            <mass value="1"/>
-            <inertia ixx="0.01" ixy="0.0" ixz="0.0" iyy="0.01" iyz="0.0" izz="0.01"/>
-        </inertial>
-        <visual>
-            <origin xyz="0 0 0" rpy="0 0 0" />
-            <geometry>
-                <cylinder length="0.3" radius="0.01" />
-            </geometry>
-            <material name="chair_metal" />
-        </visual>
-        <collision>
-            <origin xyz="0 0 0" rpy="0 0 0" />
-            <geometry>
-                <cylinder length="0.3" radius="0.01" />
-            </geometry>
-        </collision>
-    </link>
-    <!-- Chair Joints -->
-    <joint name="chair_seat_joint" type="fixed">
-        <origin xyz="0 0 0.15" rpy="0 0 0" />
-        <parent link="base_link"/>
-        <child link="chair_seat"/>
-    </joint>
-    <joint name="chair_back_joint" type="fixed">
-        <origin xyz="0.15 0 0.35" rpy="0 0 0" />
-        <parent link="chair_seat"/>
-        <child link="chair_back"/>
-    </joint>
-    <joint name="chair_leg1_joint" type="fixed">
-        <origin xyz="0.15 0.15 0.15" rpy="0 0 0" />
-        <parent link="base_link"/>
-        <child link="chair_leg1"/>
-    </joint>
-    <joint name="chair_leg2_joint" type="fixed">
-        <origin xyz="0.15 -0.15 0.15" rpy="0 0 0" />
-        <parent link="base_link"/>
-        <child link="chair_leg2"/>
-    </joint>
-    <joint name="chair_leg3_joint" type="fixed">
-        <origin xyz="-0.15 0.15 0.15" rpy="0 0 0" />
-        <parent link="base_link"/>
-        <child link="chair_leg3"/>
-    </joint>
-    <joint name="chair_leg4_joint" type="fixed">
-        <origin xyz="-0.15 -0.15 0.15" rpy="0 0 0" />
-        <parent link="base_link"/>
-        <child link="chair_leg4"/>
-    </joint>
 	<transmission name="fl_steering_wheel_trans">
       <type>transmission_interface/SimpleTransmission</type>
@@ -510,22 +513,4 @@
     </plugin>
   </gazebo>
-  <gazebo reference="chair_seat">
-    <material>Gazebo/Black</material>
-  </gazebo>
-  <gazebo reference="chair_back">
-    <material>Gazebo/Black</material>
-  </gazebo>
-  <gazebo reference="chair_leg1">
-    <material>Gazebo/Grey</material>
-  </gazebo>
-  <gazebo reference="chair_leg2">
-    <material>Gazebo/Grey</material>
-  </gazebo>
-  <gazebo reference="chair_leg3">
-    <material>Gazebo/Grey</material>
-  </gazebo>
-  <gazebo reference="chair_leg4">
-    <material>Gazebo/Grey</material>
-  </gazebo>
   <!-- Include accessories (3D LiDAR and camera) -->
   <xacro:include filename="$(find ranger_mini_v2_gazebo)/xacro/accessories.urdf.xacro" />
