Commit message: add controller

File: ranger_mini_v2_gazebo/xacro/accessories_bed.urdf.xacro (robot description, xacro)
@@ -2,8 +2,8 @@
 <robot xmlns:xacro="http://www.ros.org/wiki/xacro">
   <!--
-    Accessories for Ranger Mini Detector robot
+    Accessories for Ranger Mini Bed Trolley robot
     This file includes sensor mounts and configurations for:
     - Velodyne VLP-16 3D LiDAR
-    - Front camera (mounted on LiDAR top)
+    - Front camera
   -->
   <!-- Include accessory mount definitions -->
@@ -13,7 +13,7 @@
   <xacro:if value="$(optenv RANGER_LASER_3D 1)">
     <xacro:property name="mount" value="$(optenv RANGER_LASER_3D_MOUNT mid)" />
-    <xacro:property name="topic" value="$(optenv RANGER_LASER_3D_TOPIC detector/points)" />
+    <xacro:property name="topic" value="$(optenv RANGER_LASER_3D_TOPIC bed/points)" />
     <xacro:property name="tower" value="$(optenv RANGER_LASER_3D_TOWER 1)" />
-    <xacro:property name="prefix" value="$(optenv RANGER_LASER_3D_PREFIX detector_${mount})" />
+    <xacro:property name="prefix" value="$(optenv RANGER_LASER_3D_PREFIX bed_${mount})" />
     <xacro:property name="parent" value="$(optenv RANGER_LASER_3D_PARENT base_link)" />
     <xacro:property name="lidar_3d_model" value="$(optenv RANGER_LASER_3D_MODEL vlp16)" />
@@ -25,12 +25,12 @@
     </xacro:if>
   </xacro:if>
-  <!-- Front Camera - Same as source robot -->
+  <!-- Front Camera -->
   <xacro:if value="$(optenv RANGER_CAMERA 1)">
     <xacro:property name="mount" value="$(optenv RANGER_CAMERA_MOUNT front)" />
-    <xacro:property name="topic" value="$(optenv RANGER_CAMERA_TOPIC detector/image_raw)" />
-    <xacro:property name="prefix" value="$(optenv RANGER_CAMERA_PREFIX detector_${mount})" />
+    <xacro:property name="topic" value="$(optenv RANGER_CAMERA_TOPIC bed/image_raw)" />
+    <xacro:property name="prefix" value="$(optenv RANGER_CAMERA_PREFIX bed_${mount})" />
     <xacro:property name="parent" value="$(optenv RANGER_CAMERA_PARENT base_link)" />
     <xacro:property name="tilt" value="$(optenv RANGER_CAMERA_TILT 0)" />
-    <!-- Camera mount - same as source robot -->
+    <!-- Camera mount -->
     <xacro:camera_mount prefix="${prefix}" parent_link="${parent}">
       <origin xyz="0.2 0 0.01" rpy="0 0 0" />

File: ranger_mini_v2_gazebo/xacro/accessories_source.urdf.xacro (robot description, xacro)
@@ -2,8 +2,8 @@
 <robot xmlns:xacro="http://www.ros.org/wiki/xacro">
   <!--
-    Accessories for Ranger Mini Detector robot
+    Accessories for Ranger Mini X-ray Source robot
     This file includes sensor mounts and configurations for:
     - Velodyne VLP-16 3D LiDAR
-    - Front camera (mounted on LiDAR top)
+    - Front camera
   -->
   <!-- Include accessory mount definitions -->
@@ -13,7 +13,7 @@
   <xacro:if value="$(optenv RANGER_LASER_3D 1)">
     <xacro:property name="mount" value="$(optenv RANGER_LASER_3D_MOUNT mid)" />
-    <xacro:property name="topic" value="$(optenv RANGER_LASER_3D_TOPIC detector/points)" />
+    <xacro:property name="topic" value="$(optenv RANGER_LASER_3D_TOPIC source/points)" />
     <xacro:property name="tower" value="$(optenv RANGER_LASER_3D_TOWER 1)" />
-    <xacro:property name="prefix" value="$(optenv RANGER_LASER_3D_PREFIX detector_${mount})" />
+    <xacro:property name="prefix" value="$(optenv RANGER_LASER_3D_PREFIX source_${mount})" />
     <xacro:property name="parent" value="$(optenv RANGER_LASER_3D_PARENT base_link)" />
     <xacro:property name="lidar_3d_model" value="$(optenv RANGER_LASER_3D_MODEL vlp16)" />
@@ -25,12 +25,12 @@
     </xacro:if>
   </xacro:if>
-  <!-- Front Camera - Same as source robot -->
+  <!-- Front Camera -->
   <xacro:if value="$(optenv RANGER_CAMERA 1)">
     <xacro:property name="mount" value="$(optenv RANGER_CAMERA_MOUNT front)" />
-    <xacro:property name="topic" value="$(optenv RANGER_CAMERA_TOPIC detector/image_raw)" />
-    <xacro:property name="prefix" value="$(optenv RANGER_CAMERA_PREFIX detector_${mount})" />
+    <xacro:property name="topic" value="$(optenv RANGER_CAMERA_TOPIC source/image_raw)" />
+    <xacro:property name="prefix" value="$(optenv RANGER_CAMERA_PREFIX source_${mount})" />
     <xacro:property name="parent" value="$(optenv RANGER_CAMERA_PARENT base_link)" />
     <xacro:property name="tilt" value="$(optenv RANGER_CAMERA_TILT 0)" />
-    <!-- Camera mount - same as source robot -->
+    <!-- Camera mount -->
     <xacro:camera_mount prefix="${prefix}" parent_link="${parent}">
       <origin xyz="0.2 0 0.01" rpy="0 0 0" />

File: ranger_mini_v2_gazebo/xacro/ranger_mini_bed_trolly.xacro (robot description, xacro)
@@ -28,17 +28,17 @@
         <inertial>
             <origin xyz="0.0 0.0 0.0"/>
-            <mass value="10"/>
-            <inertia ixx="1" ixy="0.0" ixz="0.0" iyy="1" iyz="0.0" izz="1"/>
+            <mass value="33.75"/>
+            <inertia ixx="3.375" ixy="0.0" ixz="0.0" iyy="3.375" iyz="0.0" izz="3.375"/>
         </inertial>
         <visual>
             <origin xyz="0 0 0" rpy="1.57 0 3.14 " />
             <geometry>
-                <mesh filename="package://ranger_mini_v2/meshes/ranger_base.dae" />
-            </geometry>
-        </visual>
-        <collision>
-            <origin xyz="0 0 -0.1" rpy="0 0 0" />
-            <geometry>
-                <box size="0.5 0.35 0.2"/>
+                <mesh filename="package://ranger_mini_v2/meshes/ranger_base.dae" scale="1.5 1.5 1.5"/>
+            </geometry>
+        </visual>
+        <collision>
+            <origin xyz="0 0 -0.15" rpy="0 0 0" />
+            <geometry>
+                <box size="0.75 0.525 0.3"/>
             </geometry>
         </collision>
@@ -66,5 +66,5 @@
     </link>
     <joint name="bed_support_joint" type="fixed">
-        <origin xyz="-0.2 0 0" rpy="0 0 0" />
+        <origin xyz="-0.2 0 0.15" rpy="0 0 0" />
         <parent link="base_link"/>
         <child link="bed_support_link"/>
@@ -148,55 +148,4 @@
         <child link="bed_headboard_link"/>
     </joint>
-    <!-- Bed side rails -->
-    <link name="bed_rail_left_link">
-        <inertial>
-            <origin xyz="0.0 0.0 0.0"/>
-            <mass value="2"/>
-            <inertia ixx="0.05" ixy="0.0" ixz="0.0" iyy="0.05" iyz="0.0" izz="0.05"/>
-        </inertial>
-        <visual>
-            <origin xyz="0 0 0" rpy="0 0 0" />
-            <geometry>
-                <box size="1.8 0.03 0.3"/>
-            </geometry>
-            <material name="bed_metal"/>
-        </visual>
-        <collision>
-            <origin xyz="0 0 0" rpy="0 0 0" />
-            <geometry>
-                <box size="1.8 0.03 0.3"/>
-            </geometry>
-        </collision>
-    </link>
-    <joint name="bed_rail_left_joint" type="fixed">
-        <origin xyz="0 -0.415 0.15" rpy="0 0 0" />
-        <parent link="bed_frame_link"/>
-        <child link="bed_rail_left_link"/>
-    </joint>
-    <link name="bed_rail_right_link">
-        <inertial>
-            <origin xyz="0.0 0.0 0.0"/>
-            <mass value="2"/>
-            <inertia ixx="0.05" ixy="0.0" ixz="0.0" iyy="0.05" iyz="0.0" izz="0.05"/>
-        </inertial>
-        <visual>
-            <origin xyz="0 0 0" rpy="0 0 0" />
-            <geometry>
-                <box size="1.8 0.03 0.3"/>
-            </geometry>
-            <material name="bed_metal"/>
-        </visual>
-        <collision>
-            <origin xyz="0 0 0" rpy="0 0 0" />
-            <geometry>
-                <box size="1.8 0.03 0.3"/>
-            </geometry>
-        </collision>
-    </link>
-    <joint name="bed_rail_right_joint" type="fixed">
-        <origin xyz="0 0.415 0.15" rpy="0 0 0" />
-        <parent link="bed_frame_link"/>
-        <child link="bed_rail_right_link"/>
-    </joint>
    <link name="fl_steering_wheel_link">
         <inertial>
@@ -225,5 +174,5 @@
     </link>
     <joint name="fl_steering_wheel" type="revolute">
-        <origin xyz="0.23 0.206 -0.1" rpy="0 0 0" />
+        <origin xyz="0.345 0.309 -0.15" rpy="0 0 0" />
         <parent link="base_link"/>
         <child link="fl_steering_wheel_link"/>
@@ -256,5 +205,5 @@
         </link>
         <joint name="fl_wheel" type="continuous">
-            <origin xyz="0.03 0.01 -0.12" rpy="0 0 0" />
+            <origin xyz="0.045 0.015 -0.18" rpy="0 0 0" />
             <parent link="fl_steering_wheel_link"/>
             <child link="fl_wheel_link"/>
@@ -281,5 +230,5 @@
     </link>
     <joint name="fr_steering_wheel" type="revolute">
-        <origin xyz="0.23 -0.206 -0.1" rpy="0 0 0" />
+        <origin xyz="0.345 -0.309 -0.15" rpy="0 0 0" />
         <parent link="base_link"/>
         <child link="fr_steering_wheel_link"/>
@@ -312,5 +261,5 @@
         </link>
         <joint name="fr_wheel" type="continuous">
-            <origin xyz="0.0 0.0 -0.12" rpy="0 0 0" />
+            <origin xyz="0.0 0.0 -0.18" rpy="0 0 0" />
             <parent link="fr_steering_wheel_link"/>
             <child link="fr_wheel_link"/>
@@ -337,5 +286,5 @@
     </link>
     <joint name="rl_steering_wheel" type="revolute">
-        <origin xyz="-0.23 0.206 -0.1" rpy="0 0 0" />
+        <origin xyz="-0.345 0.309 -0.15" rpy="0 0 0" />
         <parent link="base_link"/>
         <child link="rl_steering_wheel_link"/>
@@ -368,5 +317,5 @@
         </link>
         <joint name="rl_wheel" type="continuous">
-            <origin xyz="0.0 0.0 -0.12 " rpy="0 0 0" />
+            <origin xyz="0.0 0.0 -0.18" rpy="0 0 0" />
             <parent link="rl_steering_wheel_link"/>
             <child link="rl_wheel_link"/>
@@ -393,5 +342,5 @@
     </link>
     <joint name="rr_steering_wheel" type="revolute">
-        <origin xyz="-0.23 -0.206 -0.1" rpy="0 0 0" />
+        <origin xyz="-0.345 -0.309 -0.15" rpy="0 0 0" />
         <parent link="base_link"/>
         <child link="rr_steering_wheel_link"/>
@@ -424,5 +373,5 @@
         </link>
         <joint name="rr_wheel" type="continuous">
-            <origin xyz="0.0 0.0 -0.12 " rpy="0 0 0" />
+            <origin xyz="0.0 0.0 -0.18" rpy="0 0 0" />
             <parent link="rr_steering_wheel_link"/>
             <child link="rr_wheel_link"/>
@@ -509,9 +458,12 @@
       </actuator>
 	</transmission>
+  <!-- Include accessories (3D LiDAR and camera) -->
+  <xacro:include filename="$(find ranger_mini_v2_gazebo)/xacro/accessories_bed.urdf.xacro" />
+  <!-- Gazebo ROS Control Plugin -->
   <gazebo>
     <plugin name="gazebo_ros_control" filename="libgazebo_ros_control.so">
+      <robotNamespace>/</robotNamespace>
+      <robotSimType>gazebo_ros_control/DefaultRobotHWSim</robotSimType>
     </plugin>
   </gazebo>
-  <!-- Include accessories (3D LiDAR and camera) -->
-  <xacro:include filename="$(find ranger_mini_v2_gazebo)/xacro/accessories.urdf.xacro" />
 </robot>

File: ranger_mini_v2_gazebo/xacro/ranger_mini_xray_detector.xacro (robot description, xacro)
@@ -454,8 +454,4 @@
       </actuator>
 	</transmission>
-  <gazebo>
-    <plugin name="gazebo_ros_control" filename="libgazebo_ros_control.so">
-    </plugin>
-  </gazebo>
   <gazebo reference="detector_board">
     <material>Gazebo/Blue</material>
@@ -466,3 +462,7 @@
   <!-- Include accessories (3D LiDAR and camera) -->
   <xacro:include filename="$(find ranger_mini_v2_gazebo)/xacro/accessories_detector.urdf.xacro" />
+  <gazebo>
+    <plugin name="gazebo_ros_control" filename="libgazebo_ros_control.so">
+    </plugin>
+  </gazebo>
 </robot>

File: ranger_mini_v2_gazebo/xacro/ranger_mini_xray_source.xacro (robot description, xacro)
@@ -345,9 +345,9 @@
       </actuator>
 	</transmission>
+  <!-- Include accessories (3D LiDAR and camera) -->
+  <xacro:include filename="$(find ranger_mini_v2_gazebo)/xacro/accessories_source.urdf.xacro" />
   <gazebo>
     <plugin name="gazebo_ros_control" filename="libgazebo_ros_control.so">
     </plugin>
   </gazebo>
-  <!-- Include accessories (3D LiDAR and camera) -->
-  <xacro:include filename="$(find ranger_mini_v2_gazebo)/xacro/accessories.urdf.xacro" />
 </robot>
