Commit message: fixed some bug

File: ranger_mini_v2_gazebo/xacro/ranger_mini_bed_trolly.xacro (robot description, xacro)
@@ -26,19 +26,15 @@
     <!-- Base link -->
     <link name="base_link">
-        <inertial>
-            <origin xyz="0.0 0.0 0.0"/>
-            <mass value="33.75"/>
-            <inertia ixx="3.375" ixy="0.0" ixz="0.0" iyy="3.375" iyz="0.0" izz="3.375"/>
-        </inertial>
         <visual>
             <origin xyz="0 0 0" rpy="1.57 0 3.14 " />
             <geometry>
-                <mesh filename="package://ranger_mini_v2/meshes/ranger_base.dae" scale="1.5 1.5 1.5"/>
-            </geometry>
-        </visual>
-        <collision>
-            <origin xyz="0 0 -0.15" rpy="0 0 0" />
-            <geometry>
-                <box size="0.75 0.525 0.3"/>
+                <mesh filename="package://ranger_mini_v2/meshes/ranger_base.dae" />
+            </geometry>
+            <material name="metallic_grey" />
+        </visual>
+        <collision>
+            <origin xyz="0 0 -0.1" rpy="0 0 0" />
+            <geometry>
+                <box size="0.6 0.45 0.25"/>
             </geometry>
         </collision>
@@ -151,11 +147,11 @@
         <inertial>
             <origin xyz="0.0 0.0 0.0"/>
-            <mass value="1"/>
-            <inertia ixx="0.01" ixy="0.0" ixz="0.0" iyy="0.01" iyz="0.0" izz="0.01"/>
-        </inertial>
-        <visual>
-            <origin xyz="-0.23 -0.194 0.1" rpy="-3.14 0 3.14 " />
-            <geometry>
-                    <mesh filename="package://ranger_mini_v2/meshes/fl.stl" />
+            <mass value="0.1"/>
+            <inertia ixx="0.001" ixy="0.0" ixz="0.0" iyy="0.001" iyz="0.0" izz="0.001"/>
+        </inertial>
+        <visual>
+            <origin xyz="0 0 0" rpy="1.57 0 3.14 " />
+            <geometry>
+                <cylinder radius="0.001" length="0.001"/>
             </geometry>
         </visual>
@@ -163,5 +159,5 @@
             <origin xyz="0 0 0.008" rpy="0 0 0" />
             <geometry>
-                <cylinder radius="0.001" length="0.001"/>
+                <box size="1 1 1"/>
             </geometry>
         </collision>
@@ -174,5 +170,5 @@
     </link>
     <joint name="fl_steering_wheel" type="revolute">
-        <origin xyz="0.345 0.309 -0.15" rpy="0 0 0" />
+        <origin xyz="0.23 0.206 -0.1" rpy="0 0 0" />
         <parent link="base_link"/>
         <child link="fl_steering_wheel_link"/>
@@ -187,13 +183,14 @@
             </inertial>
             <visual>
-                <origin xyz="0 0 0" rpy="1.57 0 0" />
-                <geometry>
-                    <cylinder length="0.01" radius="0.01" />
-                </geometry>
+                <origin xyz="0.23 -0.2 0.1" rpy="-3.14 0 0" />
+                <geometry>
+                    <mesh filename="package://ranger_mini_v2/meshes/fr.stl" />
+                </geometry>
+                <material name="black" />
             </visual>
             <collision>
-                <origin xyz="0 0 0" rpy="1.57 0 0" />
-                <geometry>
-                    <cylinder length="0.08" radius="0.08" />
+                <origin xyz="0 0 0" rpy="0 0 0" />
+                <geometry>
+                    <cylinder length="0.1" radius="0.1" />
                 </geometry>
                      <contact>
@@ -205,19 +202,19 @@
         </link>
         <joint name="fl_wheel" type="continuous">
-            <origin xyz="0.045 0.015 -0.18" rpy="0 0 0" />
+            <origin xyz="0.0 0.0 0.0" rpy="0 0 0" />
             <parent link="fl_steering_wheel_link"/>
             <child link="fl_wheel_link"/>
-            <axis xyz="0 1 0" rpy="0 0 0" />
+            <axis xyz="0 0 1" rpy="0 0 0" />
         </joint>
    <link name="fr_steering_wheel_link">
         <inertial>
-            <origin xyz="0.0 0.0 0.0" rpy="0.0 0.0 0.0"/>
-            <mass value="1"/>
-            <inertia ixx="0.01" ixy="0.0" ixz="0.0" iyy="0.01" iyz="0.0" izz="0.01"/>
-        </inertial>
-        <visual>
-            <origin xyz="-0.23 0.194 0.1" rpy="-3.14 0 3.14 " />
-            <geometry>
-                <mesh filename="package://ranger_mini_v2/meshes/fr.stl" />
+            <origin xyz="0.0 0.0 0.0"/>
+            <mass value="0.1"/>
+            <inertia ixx="0.001" ixy="0.0" ixz="0.0" iyy="0.001" iyz="0.0" izz="0.001"/>
+        </inertial>
+        <visual>
+            <origin xyz="0 0 0" rpy="1.57 0 3.14 " />
+            <geometry>
+                <cylinder radius="0.001" length="0.001"/>
             </geometry>
         </visual>
@@ -225,4 +222,10 @@
             <origin xyz="0 0 0.008" rpy="0 0 0" />
             <geometry>
+                <box size="1 1 1"/>
+            </geometry>
+        </collision>
+        <collision>
+            <origin xyz="0 0 0" rpy="0 0 0" />
+            <geometry>
                 <cylinder radius="0.001" length="0.001"/>
             </geometry>
@@ -230,5 +233,5 @@
     </link>
     <joint name="fr_steering_wheel" type="revolute">
-        <origin xyz="0.345 -0.309 -0.15" rpy="0 0 0" />
+        <origin xyz="0.23 -0.206 -0.1" rpy="0 0 0" />
         <parent link="base_link"/>
         <child link="fr_steering_wheel_link"/>
@@ -243,13 +246,14 @@
             </inertial>
             <visual>
-                <origin xyz="0 0 0" rpy="1.57 0 0" />
-                <geometry>
-                    <cylinder length="0.01" radius="0.01" />
-                </geometry>
+                <origin xyz="0.23 0.2 0.1" rpy="-3.14 0 0" />
+                <geometry>
+                    <mesh filename="package://ranger_mini_v2/meshes/fl.stl" />
+                </geometry>
+                <material name="black" />
             </visual>
             <collision>
-                <origin xyz="0 0 0" rpy="1.57 0 0" />
-                <geometry>
-                    <cylinder length="0.08" radius="0.085" />
+                <origin xyz="0 0 0" rpy="0 0 0" />
+                <geometry>
+                    <cylinder length="0.1" radius="0.1" />
                 </geometry>
                      <contact>
@@ -261,19 +265,19 @@
         </link>
         <joint name="fr_wheel" type="continuous">
-            <origin xyz="0.0 0.0 -0.18" rpy="0 0 0" />
+            <origin xyz="0.0 0.0 0.0" rpy="0 0 0" />
             <parent link="fr_steering_wheel_link"/>
             <child link="fr_wheel_link"/>
-            <axis xyz="0 1 0" rpy="0 0 0" />
+            <axis xyz="0 0 1" rpy="0 0 0" />
         </joint>
    <link name="rl_steering_wheel_link">
         <inertial>
-            <origin xyz="0.0 0.0 0.0" rpy="0.0 0.0 0.0"/>
-            <mass value="1"/>
-            <inertia ixx="0.01" ixy="0.0" ixz="0.0" iyy="0.01" iyz="0.0" izz="0.01"/>
-        </inertial>
-        <visual>
-            <origin xyz="-0.23 -0.194 0.1" rpy="-3.14 0 3.14 " />
-            <geometry>
-                    <mesh filename="package://ranger_mini_v2/meshes/fl.stl" />
+            <origin xyz="0.0 0.0 0.0"/>
+            <mass value="0.1"/>
+            <inertia ixx="0.001" ixy="0.0" ixz="0.0" iyy="0.001" iyz="0.0" izz="0.001"/>
+        </inertial>
+        <visual>
+            <origin xyz="0 0 0" rpy="1.57 0 3.14 " />
+            <geometry>
+                <cylinder radius="0.001" length="0.001"/>
             </geometry>
         </visual>
@@ -281,4 +285,10 @@
             <origin xyz="0 0 0.008" rpy="0 0 0" />
             <geometry>
+                <box size="1 1 1"/>
+            </geometry>
+        </collision>
+        <collision>
+            <origin xyz="0 0 0" rpy="0 0 0" />
+            <geometry>
                 <cylinder radius="0.001" length="0.001"/>
             </geometry>
@@ -286,5 +296,5 @@
     </link>
     <joint name="rl_steering_wheel" type="revolute">
-        <origin xyz="-0.345 0.309 -0.15" rpy="0 0 0" />
+        <origin xyz="-0.23 0.206 -0.1" rpy="0 0 0" />
         <parent link="base_link"/>
         <child link="rl_steering_wheel_link"/>
@@ -299,13 +309,14 @@
             </inertial>
             <visual>
-                <origin xyz="0 0 0" rpy="1.57 0 0" />
-                <geometry>
-                    <cylinder length="0.01" radius="0.01" />
-                </geometry>
+                <origin xyz="0.23 -0.2 0.1" rpy="-3.14 0 0" />
+                <geometry>
+                    <mesh filename="package://ranger_mini_v2/meshes/fr.stl" />
+                </geometry>
+                <material name="black" />
             </visual>
             <collision>
-                <origin xyz="0 0 0" rpy="1.57 0 0" />
-                <geometry>
-                    <cylinder length="0.08" radius="0.08" />
+                <origin xyz="0 0 0" rpy="0 0 0" />
+                <geometry>
+                    <cylinder length="0.1" radius="0.1" />
                 </geometry>
                      <contact>
@@ -317,21 +328,27 @@
         </link>
         <joint name="rl_wheel" type="continuous">
-            <origin xyz="0.0 0.0 -0.18" rpy="0 0 0" />
+            <origin xyz="0.0 0.0 0.0" rpy="0 0 0" />
             <parent link="rl_steering_wheel_link"/>
             <child link="rl_wheel_link"/>
-            <axis xyz="0 1 0" rpy="0 0 0" />
+            <axis xyz="0 0 1" rpy="0 0 0" />
         </joint>
    <link name="rr_steering_wheel_link">
         <inertial>
             <origin xyz="0.0 0.0 0.0"/>
-            <mass value="1"/>
-            <inertia ixx="0.01" ixy="0.0" ixz="0.0" iyy="0.01" iyz="0.0" izz="0.01"/>
-        </inertial>
-        <visual>
-            <origin xyz="-0.23 0.194 0.1" rpy="-3.14 0 3.14 " />
-            <geometry>
-                    <mesh filename="package://ranger_mini_v2/meshes/fr.stl" />
-            </geometry>
-        </visual>
+            <mass value="0.1"/>
+            <inertia ixx="0.001" ixy="0.0" ixz="0.0" iyy="0.001" iyz="0.0" izz="0.001"/>
+        </inertial>
+        <visual>
+            <origin xyz="0 0 0" rpy="1.57 0 3.14 " />
+            <geometry>
+                <cylinder radius="0.001" length="0.001"/>
+            </geometry>
+        </visual>
+        <collision>
+            <origin xyz="0 0 0.008" rpy="0 0 0" />
+            <geometry>
+                <box size="1 1 1"/>
+            </geometry>
+        </collision>
         <collision>
             <origin xyz="0 0 0" rpy="0 0 0" />
@@ -342,5 +359,5 @@
     </link>
     <joint name="rr_steering_wheel" type="revolute">
-        <origin xyz="-0.345 -0.309 -0.15" rpy="0 0 0" />
+        <origin xyz="-0.23 -0.206 -0.1" rpy="0 0 0" />
         <parent link="base_link"/>
         <child link="rr_steering_wheel_link"/>
@@ -355,13 +372,14 @@
             </inertial>
             <visual>
-                <origin xyz="0.0 0.0 0.0" rpy="1.57 0 0" />
-                <geometry>
-                    <cylinder length="0.01" radius="0.01" />
-                </geometry>
+                <origin xyz="0.23 0.2 0.1" rpy="-3.14 0 0" />
+                <geometry>
+                    <mesh filename="package://ranger_mini_v2/meshes/fl.stl" />
+                </geometry>
+                <material name="black" />
             </visual>
             <collision>
-                <origin xyz="0 0 0" rpy="1.57 0 0" />
-                <geometry>
-                    <cylinder length="0.08" radius="0.08" />
+                <origin xyz="0 0 0" rpy="0 0 0" />
+                <geometry>
+                    <cylinder length="0.1" radius="0.1" />
                 </geometry>
                      <contact>
@@ -373,8 +391,8 @@
         </link>
         <joint name="rr_wheel" type="continuous">
-            <origin xyz="0.0 0.0 -0.18" rpy="0 0 0" />
+            <origin xyz="0.0 0.0 0.0" rpy="0 0 0" />
             <parent link="rr_steering_wheel_link"/>
             <child link="rr_wheel_link"/>
-            <axis xyz="0 1 0" rpy="0 0 0" />
+            <axis xyz="0 0 1" rpy="0 0 0" />
         </joint>
 	<transmission name="fl_steering_wheel_trans">

File: ranger_mini_v2_gazebo/xacro/ranger_mini_xray_detector.xacro (robot description, xacro)
@@ -20,9 +20,4 @@
     <!-- Base link -->
     <link name="base_link">
-        <inertial>
-            <origin xyz="0.0 0.0 0.0"/>
-            <mass value="10"/>
-            <inertia ixx="1" ixy="0.0" ixz="0.0" iyy="1" iyz="0.0" izz="1"/>
-        </inertial>
         <visual>
             <origin xyz="0 0 0" rpy="1.57 0 3.14 " />
@@ -30,4 +25,5 @@
                 <mesh filename="package://ranger_mini_v2/meshes/ranger_base.dae" />
             </geometry>
+            <material name="metallic_grey" />
         </visual>
         <collision>
@@ -49,4 +45,5 @@
                     <mesh filename="package://ranger_mini_v2/meshes/fl.stl" />
             </geometry>
+            <material name="dark_grey" />
         </visual>
         <collision>
@@ -81,4 +78,5 @@
                     <cylinder length="0.01" radius="0.01" />
                 </geometry>
+                <material name="black" />
             </visual>
             <collision>
@@ -111,4 +109,5 @@
                 <mesh filename="package://ranger_mini_v2/meshes/fr.stl" />
             </geometry>
+            <material name="dark_grey" />
         </visual>
         <collision>
@@ -137,4 +136,5 @@
                     <cylinder length="0.01" radius="0.01" />
                 </geometry>
+                <material name="black" />
             </visual>
             <collision>
@@ -167,4 +167,5 @@
                     <mesh filename="package://ranger_mini_v2/meshes/fl.stl" />
             </geometry>
+            <material name="dark_grey" />
         </visual>
         <collision>
@@ -193,4 +194,5 @@
                     <cylinder length="0.01" radius="0.01" />
                 </geometry>
+                <material name="black" />
             </visual>
             <collision>
@@ -223,4 +225,5 @@
                     <mesh filename="package://ranger_mini_v2/meshes/fr.stl" />
             </geometry>
+            <material name="dark_grey" />
         </visual>
         <collision>
@@ -249,4 +252,5 @@
                     <cylinder length="0.01" radius="0.01" />
                 </geometry>
+                <material name="black" />
             </visual>
             <collision>
@@ -462,6 +466,9 @@
   <!-- Include accessories (3D LiDAR and camera) -->
   <xacro:include filename="$(find ranger_mini_v2_gazebo)/xacro/accessories_detector.urdf.xacro" />
+  <!-- Gazebo ROS Control Plugin -->
   <gazebo>
     <plugin name="gazebo_ros_control" filename="libgazebo_ros_control.so">
+      <robotNamespace>/</robotNamespace>
+      <robotSimType>gazebo_ros_control/DefaultRobotHWSim</robotSimType>
     </plugin>
   </gazebo>

File: ranger_mini_v2_gazebo/xacro/ranger_mini_xray_source.xacro (robot description, xacro)
@@ -15,11 +15,9 @@
         <color rgba="0.7 0.7 0.7 1" />
     </material>
+    <material name="source_red">
+        <color rgba="0.8 0.2 0.2 1" />
+    </material>
     <!-- Base link -->
     <link name="base_link">
-        <inertial>
-            <origin xyz="0.0 0.0 0.0"/>
-            <mass value="10"/>
-            <inertia ixx="1" ixy="0.0" ixz="0.0" iyy="1" iyz="0.0" izz="1"/>
-        </inertial>
         <visual>
             <origin xyz="0 0 0" rpy="1.57 0 3.14 " />
@@ -27,4 +25,5 @@
                 <mesh filename="package://ranger_mini_v2/meshes/ranger_base.dae" />
             </geometry>
+            <material name="metallic_grey" />
         </visual>
         <collision>
@@ -46,4 +45,5 @@
                     <mesh filename="package://ranger_mini_v2/meshes/fl.stl" />
             </geometry>
+            <material name="dark_grey" />
         </visual>
         <collision>
@@ -78,4 +78,5 @@
                     <cylinder length="0.01" radius="0.01" />
                 </geometry>
+                <material name="black" />
             </visual>
             <collision>
@@ -108,4 +109,5 @@
                 <mesh filename="package://ranger_mini_v2/meshes/fr.stl" />
             </geometry>
+            <material name="dark_grey" />
         </visual>
         <collision>
@@ -134,4 +136,5 @@
                     <cylinder length="0.01" radius="0.01" />
                 </geometry>
+                <material name="black" />
             </visual>
             <collision>
@@ -164,4 +167,5 @@
                     <mesh filename="package://ranger_mini_v2/meshes/fl.stl" />
             </geometry>
+            <material name="dark_grey" />
         </visual>
         <collision>
@@ -190,4 +194,5 @@
                     <cylinder length="0.01" radius="0.01" />
                 </geometry>
+                <material name="black" />
             </visual>
             <collision>
@@ -220,4 +225,5 @@
                     <mesh filename="package://ranger_mini_v2/meshes/fr.stl" />
             </geometry>
+            <material name="dark_grey" />
         </visual>
         <collision>
@@ -246,4 +252,5 @@
                     <cylinder length="0.01" radius="0.01" />
                 </geometry>
+                <material name="black" />
             </visual>
             <collision>
@@ -347,6 +354,9 @@
   <!-- Include accessories (3D LiDAR and camera) -->
   <xacro:include filename="$(find ranger_mini_v2_gazebo)/xacro/accessories_source.urdf.xacro" />
+  <!-- Gazebo ROS Control Plugin -->
   <gazebo>
     <plugin name="gazebo_ros_control" filename="libgazebo_ros_control.so">
+      <robotNamespace>/</robotNamespace>
+      <robotSimType>gazebo_ros_control/DefaultRobotHWSim</robotSimType>
     </plugin>
   </gazebo>
