Commit message: fix model

File: ranger_mini_v2_gazebo/xacro/ranger_mini_bed_trolly.xacro (robot description, xacro)
@@ -26,4 +26,9 @@
     <!-- Base link -->
     <link name="base_link">
+        <inertial>
+            <origin xyz="0.0 0.0 0.0"/>
+            <mass value="20"/>
+            <inertia ixx="0.8" ixy="0.0" ixz="0.0" iyy="0.8" iyz="0.0" izz="0.8"/>
+        </inertial>
         <visual>
             <origin xyz="0 0 0" rpy="1.57 0 3.14 " />
@@ -147,17 +152,18 @@
         <inertial>
             <origin xyz="0.0 0.0 0.0"/>
-            <mass value="0.1"/>
-            <inertia ixx="0.001" ixy="0.0" ixz="0.0" iyy="0.001" iyz="0.0" izz="0.001"/>
-        </inertial>
-        <visual>
-            <origin xyz="0 0 0" rpy="1.57 0 3.14 " />
+            <mass value="1"/>
+            <inertia ixx="0.01" ixy="0.0" ixz="0.0" iyy="0.01" iyz="0.0" izz="0.01"/>
+        </inertial>
+        <visual>
+            <origin xyz="-0.23 -0.194 0.1" rpy="-3.14 0 3.14 " />
+            <geometry>
+                    <mesh filename="package://ranger_mini_v2/meshes/fl.stl" />
+            </geometry>
+            <material name="dark_grey" />
+        </visual>
+        <collision>
+            <origin xyz="0 0 0.008" rpy="0 0 0" />
             <geometry>
                 <cylinder radius="0.001" length="0.001"/>
-            </geometry>
-        </visual>
-        <collision>
-            <origin xyz="0 0 0.008" rpy="0 0 0" />
-            <geometry>
-                <box size="1 1 1"/>
             </geometry>
         </collision>
@@ -183,14 +189,14 @@
             </inertial>
             <visual>
-                <origin xyz="0.23 -0.2 0.1" rpy="-3.14 0 0" />
-                <geometry>
-                    <mesh filename="package://ranger_mini_v2/meshes/fr.stl" />
+                <origin xyz="0 0 0" rpy="1.57 0 0" />
+                <geometry>
+                    <cylinder length="0.01" radius="0.01" />
                 </geometry>
                 <material name="black" />
             </visual>
             <collision>
-                <origin xyz="0 0 0" rpy="0 0 0" />
-                <geometry>
-                    <cylinder length="0.1" radius="0.1" />
+                <origin xyz="0 0 0" rpy="1.57 0 0" />
+                <geometry>
+                    <cylinder length="0.08" radius="0.08" />
                 </geometry>
                      <contact>
@@ -202,29 +208,24 @@
         </link>
         <joint name="fl_wheel" type="continuous">
-            <origin xyz="0.0 0.0 0.0" rpy="0 0 0" />
+            <origin xyz="0.03 0.01 -0.12" rpy="0 0 0" />
             <parent link="fl_steering_wheel_link"/>
             <child link="fl_wheel_link"/>
-            <axis xyz="0 0 1" rpy="0 0 0" />
+            <axis xyz="0 1 0" rpy="0 0 0" />
         </joint>
    <link name="fr_steering_wheel_link">
         <inertial>
-            <origin xyz="0.0 0.0 0.0"/>
-            <mass value="0.1"/>
-            <inertia ixx="0.001" ixy="0.0" ixz="0.0" iyy="0.001" iyz="0.0" izz="0.001"/>
-        </inertial>
-        <visual>
-            <origin xyz="0 0 0" rpy="1.57 0 3.14 " />
-            <geometry>
-                <cylinder radius="0.001" length="0.001"/>
-            </geometry>
+            <origin xyz="0.0 0.0 0.0" rpy="0.0 0.0 0.0"/>
+            <mass value="1"/>
+            <inertia ixx="0.01" ixy="0.0" ixz="0.0" iyy="0.01" iyz="0.0" izz="0.01"/>
+        </inertial>
+        <visual>
+            <origin xyz="-0.23 0.194 0.1" rpy="-3.14 0 3.14 " />
+            <geometry>
+                <mesh filename="package://ranger_mini_v2/meshes/fr.stl" />
+            </geometry>
+            <material name="dark_grey" />
         </visual>
         <collision>
             <origin xyz="0 0 0.008" rpy="0 0 0" />
-            <geometry>
-                <box size="1 1 1"/>
-            </geometry>
-        </collision>
-        <collision>
-            <origin xyz="0 0 0" rpy="0 0 0" />
             <geometry>
                 <cylinder radius="0.001" length="0.001"/>
@@ -246,14 +247,14 @@
             </inertial>
             <visual>
-                <origin xyz="0.23 0.2 0.1" rpy="-3.14 0 0" />
-                <geometry>
-                    <mesh filename="package://ranger_mini_v2/meshes/fl.stl" />
+                <origin xyz="0 0 0" rpy="1.57 0 0" />
+                <geometry>
+                    <cylinder length="0.01" radius="0.01" />
                 </geometry>
                 <material name="black" />
             </visual>
             <collision>
-                <origin xyz="0 0 0" rpy="0 0 0" />
-                <geometry>
-                    <cylinder length="0.1" radius="0.1" />
+                <origin xyz="0 0 0" rpy="1.57 0 0" />
+                <geometry>
+                    <cylinder length="0.08" radius="0.085" />
                 </geometry>
                      <contact>
@@ -265,29 +266,24 @@
         </link>
         <joint name="fr_wheel" type="continuous">
-            <origin xyz="0.0 0.0 0.0" rpy="0 0 0" />
+            <origin xyz="0.0 0.0 -0.12" rpy="0 0 0" />
             <parent link="fr_steering_wheel_link"/>
             <child link="fr_wheel_link"/>
-            <axis xyz="0 0 1" rpy="0 0 0" />
+            <axis xyz="0 1 0" rpy="0 0 0" />
         </joint>
    <link name="rl_steering_wheel_link">
         <inertial>
-            <origin xyz="0.0 0.0 0.0"/>
-            <mass value="0.1"/>
-            <inertia ixx="0.001" ixy="0.0" ixz="0.0" iyy="0.001" iyz="0.0" izz="0.001"/>
-        </inertial>
-        <visual>
-            <origin xyz="0 0 0" rpy="1.57 0 3.14 " />
-            <geometry>
-                <cylinder radius="0.001" length="0.001"/>
-            </geometry>
+            <origin xyz="0.0 0.0 0.0" rpy="0.0 0.0 0.0"/>
+            <mass value="1"/>
+            <inertia ixx="0.01" ixy="0.0" ixz="0.0" iyy="0.01" iyz="0.0" izz="0.01"/>
+        </inertial>
+        <visual>
+            <origin xyz="-0.23 -0.194 0.1" rpy="-3.14 0 3.14 " />
+            <geometry>
+                    <mesh filename="package://ranger_mini_v2/meshes/fl.stl" />
+            </geometry>
+            <material name="dark_grey" />
         </visual>
         <collision>
             <origin xyz="0 0 0.008" rpy="0 0 0" />
-            <geometry>
-                <box size="1 1 1"/>
-            </geometry>
-        </collision>
-        <collision>
-            <origin xyz="0 0 0" rpy="0 0 0" />
             <geometry>
                 <cylinder radius="0.001" length="0.001"/>
@@ -309,14 +305,14 @@
             </inertial>
             <visual>
-                <origin xyz="0.23 -0.2 0.1" rpy="-3.14 0 0" />
-                <geometry>
-                    <mesh filename="package://ranger_mini_v2/meshes/fr.stl" />
+                <origin xyz="0 0 0" rpy="1.57 0 0" />
+                <geometry>
+                    <cylinder length="0.01" radius="0.01" />
                 </geometry>
                 <material name="black" />
             </visual>
             <collision>
-                <origin xyz="0 0 0" rpy="0 0 0" />
-                <geometry>
-                    <cylinder length="0.1" radius="0.1" />
+                <origin xyz="0 0 0" rpy="1.57 0 0" />
+                <geometry>
+                    <cylinder length="0.08" radius="0.08" />
                 </geometry>
                      <contact>
@@ -328,29 +324,24 @@
         </link>
         <joint name="rl_wheel" type="continuous">
-            <origin xyz="0.0 0.0 0.0" rpy="0 0 0" />
+            <origin xyz="0.03 0.01 -0.12" rpy="0 0 0" />
             <parent link="rl_steering_wheel_link"/>
             <child link="rl_wheel_link"/>
-            <axis xyz="0 0 1" rpy="0 0 0" />
+            <axis xyz="0 1 0" rpy="0 0 0" />
         </joint>
    <link name="rr_steering_wheel_link">
         <inertial>
-            <origin xyz="0.0 0.0 0.0"/>
-            <mass value="0.1"/>
-            <inertia ixx="0.001" ixy="0.0" ixz="0.0" iyy="0.001" iyz="0.0" izz="0.001"/>
-        </inertial>
-        <visual>
-            <origin xyz="0 0 0" rpy="1.57 0 3.14 " />
-            <geometry>
-                <cylinder radius="0.001" length="0.001"/>
-            </geometry>
+            <origin xyz="0.0 0.0 0.0" rpy="0.0 0.0 0.0"/>
+            <mass value="1"/>
+            <inertia ixx="0.01" ixy="0.0" ixz="0.0" iyy="0.01" iyz="0.0" izz="0.01"/>
+        </inertial>
+        <visual>
+            <origin xyz="-0.23 0.194 0.1" rpy="-3.14 0 3.14 " />
+            <geometry>
+                    <mesh filename="package://ranger_mini_v2/meshes/fr.stl" />
+            </geometry>
+            <material name="dark_grey" />
         </visual>
         <collision>
             <origin xyz="0 0 0.008" rpy="0 0 0" />
-            <geometry>
-                <box size="1 1 1"/>
-            </geometry>
-        </collision>
-        <collision>
-            <origin xyz="0 0 0" rpy="0 0 0" />
             <geometry>
                 <cylinder radius="0.001" length="0.001"/>
@@ -372,14 +363,14 @@
             </inertial>
             <visual>
-                <origin xyz="0.23 0.2 0.1" rpy="-3.14 0 0" />
-                <geometry>
-                    <mesh filename="package://ranger_mini_v2/meshes/fl.stl" />
+                <origin xyz="0 0 0" rpy="1.57 0 0" />
+                <geometry>
+                    <cylinder length="0.01" radius="0.01" />
                 </geometry>
                 <material name="black" />
             </visual>
             <collision>
-                <origin xyz="0 0 0" rpy="0 0 0" />
-                <geometry>
-                    <cylinder length="0.1" radius="0.1" />
+                <origin xyz="0 0 0" rpy="1.57 0 0" />
+                <geometry>
+                    <cylinder length="0.08" radius="0.08" />
                 </geometry>
                      <contact>
@@ -391,8 +382,8 @@
         </link>
         <joint name="rr_wheel" type="continuous">
-            <origin xyz="0.0 0.0 0.0" rpy="0 0 0" />
+            <origin xyz="0.03 0.01 -0.12" rpy="0 0 0" />
             <parent link="rr_steering_wheel_link"/>
             <child link="rr_wheel_link"/>
-            <axis xyz="0 0 1" rpy="0 0 0" />
+            <axis xyz="0 1 0" rpy="0 0 0" />
         </joint>
 	<transmission name="fl_steering_wheel_trans">

File: ranger_mini_v2_gazebo/xacro/ranger_mini_xray_detector.xacro (robot description, xacro)
@@ -470,5 +470,5 @@
     <plugin name="gazebo_ros_control" filename="libgazebo_ros_control.so">
       <robotNamespace>/xray_detector</robotNamespace>
-      <robotParam>robot_description_xray_detector</robotParam>
+              <robotParam>robot_description</robotParam>
       <robotSimType>gazebo_ros_control/DefaultRobotHWSim</robotSimType>
     </plugin>

File: ranger_mini_v2_gazebo/xacro/ranger_mini_xray_source.xacro (robot description, xacro)
@@ -20,4 +20,9 @@
     <!-- Base link -->
     <link name="base_link">
+        <inertial>
+            <origin xyz="0.0 0.0 0.0"/>
+            <mass value="15"/>
+            <inertia ixx="0.5" ixy="0.0" ixz="0.0" iyy="0.5" iyz="0.0" izz="0.5"/>
+        </inertial>
         <visual>
             <origin xyz="0 0 0" rpy="1.57 0 3.14 " />
@@ -272,4 +277,58 @@
             <axis xyz="0 1 0" rpy="0 0 0" />
         </joint>
+    <!-- X-ray Source Component -->
+    <link name="xray_source_component">
+        <inertial>
+            <origin xyz="0.0 0.0 0.0"/>
+            <mass value="5"/>
+            <inertia ixx="0.2" ixy="0.0" ixz="0.0" iyy="0.2" iyz="0.0" izz="0.2"/>
+        </inertial>
+        <visual>
+            <origin xyz="0 0 0" rpy="0 0 0" />
+            <geometry>
+                <cylinder radius="0.1" length="0.3" />
+            </geometry>
+            <material name="source_red" />
+        </visual>
+        <collision>
+            <origin xyz="0 0 0" rpy="0 0 0" />
+            <geometry>
+                <cylinder radius="0.1" length="0.3" />
+            </geometry>
+        </collision>
+    </link>
+    <!-- X-ray Source Support -->
+    <link name="xray_source_support">
+        <inertial>
+            <origin xyz="0.0 0.0 0.0"/>
+            <mass value="2"/>
+            <inertia ixx="0.1" ixy="0.0" ixz="0.0" iyy="0.1" iyz="0.0" izz="0.1"/>
+        </inertial>
+        <visual>
+            <origin xyz="0 0 0" rpy="0 0 0" />
+            <geometry>
+                <box size="0.02 0.02 0.4" />
+            </geometry>
+            <material name="dark_grey" />
+        </visual>
+        <collision>
+            <origin xyz="0 0 0" rpy="0 0 0" />
+            <geometry>
+                <box size="0.02 0.02 0.4" />
+            </geometry>
+        </collision>
+    </link>
+    <!-- Connect source support to base -->
+    <joint name="xray_source_support_joint" type="fixed">
+        <origin xyz="0 0 0.2" rpy="0 0 0" />
+        <parent link="base_link"/>
+        <child link="xray_source_support"/>
+    </joint>
+    <!-- Connect source component to support -->
+    <joint name="xray_source_component_joint" type="fixed">
+        <origin xyz="0 0 0.4" rpy="0 0 0" />
+        <parent link="xray_source_support"/>
+        <child link="xray_source_component"/>
+    </joint>
 	<transmission name="fl_steering_wheel_trans">
       <type>transmission_interface/SimpleTransmission</type>
@@ -358,5 +417,5 @@
     <plugin name="gazebo_ros_control" filename="libgazebo_ros_control.so">
       <robotNamespace>/xray_source</robotNamespace>
-      <robotParam>robot_description_xray_source</robotParam>
+              <robotParam>robot_description</robotParam>
       <robotSimType>gazebo_ros_control/DefaultRobotHWSim</robotSimType>
     </plugin>
