Commit message: changed structure

File: ranger_mini_v2_gazebo/xacro/ranger_mini_xray_detector.xacro (robot description, xacro)
@@ -268,15 +268,15 @@
             <axis xyz="0 1 0" rpy="0 0 0" />
         </joint>
-    <!-- X-ray Detector Board - Vertical Tag-like Structure -->
-    <link name="detector_board">
+    <!-- Detector Board 1 - Connected to leg1 -->
+    <link name="detector_board1">
         <inertial>
             <origin xyz="0.0 0.0 -0.28"/>
-            <mass value="3"/>
-            <inertia ixx="0.2" ixy="0.0" ixz="0.0" iyy="0.2" iyz="0.0" izz="0.2"/>
-        </inertial>
-        <visual>
-            <origin xyz="0 0 0" rpy="0 0 0" />
-            <geometry>
-                <box size="0.8 0.02 0.6" />
+            <mass value="2"/>
+            <inertia ixx="0.15" ixy="0.0" ixz="0.0" iyy="0.15" iyz="0.0" izz="0.15"/>
+        </inertial>
+        <visual>
+            <origin xyz="0 0 0" rpy="0 0 0" />
+            <geometry>
+                <box size="0.3 0.02 0.6" />
             </geometry>
             <material name="detector_blue" />
@@ -285,19 +285,40 @@
             <origin xyz="0 0 0" rpy="0 0 0" />
             <geometry>
-                <box size="0.6 0.02 0.8" />
-            </geometry>
-        </collision>
-    </link>
-    <!-- Detector Board Support Frame - Connected to LiDAR -->
-    <link name="detector_support">
+                <box size="0.3 0.02 0.6" />
+            </geometry>
+        </collision>
+    </link>
+    <!-- Detector Board 2 - Connected to leg2 -->
+    <link name="detector_board2">
+        <inertial>
+            <origin xyz="0.0 0.0 -0.28"/>
+            <mass value="2"/>
+            <inertia ixx="0.15" ixy="0.0" ixz="0.0" iyy="0.15" iyz="0.0" izz="0.15"/>
+        </inertial>
+        <visual>
+            <origin xyz="0 0 0" rpy="0 0 0" />
+            <geometry>
+                <box size="0.3 0.02 0.6" />
+            </geometry>
+            <material name="detector_blue" />
+        </visual>
+        <collision>
+            <origin xyz="0 0 0" rpy="0 0 0" />
+            <geometry>
+                <box size="0.3 0.02 0.6" />
+            </geometry>
+        </collision>
+    </link>
+    <!-- Detector Board Support Frame - Two thin legs connected to base -->
+    <link name="detector_support_leg1">
         <inertial>
             <origin xyz="0.0 0.0 0.0"/>
-            <mass value="1"/>
-            <inertia ixx="0.05" ixy="0.0" ixz="0.0" iyy="0.05" iyz="0.0" izz="0.05"/>
-        </inertial>
-        <visual>
-            <origin xyz="0 0 0" rpy="0 0 0" />
-            <geometry>
-                <box size="0.02 0.02 0.2" />
+            <mass value="0.25"/>
+            <inertia ixx="0.01" ixy="0.0" ixz="0.0" iyy="0.01" iyz="0.0" izz="0.01"/>
+        </inertial>
+        <visual>
+            <origin xyz="0 0 0" rpy="0 0 0" />
+            <geometry>
+                <box size="0.02 0.02 0.4" />
             </geometry>
             <material name="dark_grey" />
@@ -306,17 +327,50 @@
             <origin xyz="0 0 0" rpy="0 0 0" />
             <geometry>
-                <box size="0.05 0.05 0.2" />
-            </geometry>
-        </collision>
-    </link>
-    <joint name="detector_support_joint" type="fixed">
-        <origin xyz="0 0 0.08" rpy="0 0 0" />
-        <parent link="velodyne"/>
-        <child link="detector_support"/>
-    </joint>
-    <joint name="detector_board_joint" type="fixed">
-        <origin xyz="0 0 0.32" rpy="0 0 0" />
-        <parent link="detector_support"/>
-        <child link="detector_board"/>
+                <box size="0.02 0.02 0.4" />
+            </geometry>
+        </collision>
+    </link>
+    <link name="detector_support_leg2">
+        <inertial>
+            <origin xyz="0.0 0.0 0.0"/>
+            <mass value="0.25"/>
+            <inertia ixx="0.01" ixy="0.0" ixz="0.0" iyy="0.01" iyz="0.0" izz="0.01"/>
+        </inertial>
+        <visual>
+            <origin xyz="0 0 0" rpy="0 0 0" />
+            <geometry>
+                <box size="0.02 0.02 0.4" />
+            </geometry>
+            <material name="dark_grey" />
+        </visual>
+        <collision>
+            <origin xyz="0 0 0" rpy="0 0 0" />
+            <geometry>
+                <box size="0.02 0.02 0.4" />
+            </geometry>
+        </collision>
+    </link>
+    <!-- Two support legs connected to base (front left and front right) -->
+    <joint name="detector_support_leg1_joint" type="fixed">
+        <origin xyz="0.15 0.1 0.2" rpy="0 0 0" />
+        <parent link="base_link"/>
+        <child link="detector_support_leg1"/>
+    </joint>
+    <joint name="detector_support_leg2_joint" type="fixed">
+        <origin xyz="-0.15 0.1 0.2" rpy="0 0 0" />
+        <parent link="base_link"/>
+        <child link="detector_support_leg2"/>
+    </joint>
+    <!-- Connect board1 to leg1 -->
+    <joint name="detector_board1_joint" type="fixed">
+        <origin xyz="0 0 0.4" rpy="0 0 0" />
+        <parent link="detector_support_leg1"/>
+        <child link="detector_board1"/>
+    </joint>
+    <!-- Connect board2 to leg2 -->
+    <joint name="detector_board2_joint" type="fixed">
+        <origin xyz="0 0 0.4" rpy="0 0 0" />
+        <parent link="detector_support_leg2"/>
+        <child link="detector_board2"/>
     </joint>
 	<transmission name="fl_steering_wheel_trans">

Commit message: changde mode

File: ranger_mini_v2_gazebo/xacro/ranger_mini_xray_detector.xacro (robot description, xacro)
@@ -275,12 +275,12 @@
     <link name="detector_board1">
         <inertial>
-            <origin xyz="0.0 0.0 -0.28"/>
-            <mass value="2"/>
-            <inertia ixx="0.15" ixy="0.0" ixz="0.0" iyy="0.15" iyz="0.0" izz="0.15"/>
-        </inertial>
-        <visual>
-            <origin xyz="0 0 0" rpy="0 0 0" />
-            <geometry>
-                <box size="0.3 0.02 0.6" />
+            <origin xyz="0.0 0.0 -0.35"/>
+            <mass value="3"/>
+            <inertia ixx="0.2" ixy="0.0" ixz="0.0" iyy="0.2" iyz="0.0" izz="0.2"/>
+        </inertial>
+        <visual>
+            <origin xyz="0 0 0" rpy="0 0 0" />
+            <geometry>
+                <box size="0.4 0.03 0.8" />
             </geometry>
             <material name="detector_blue" />
@@ -289,5 +289,5 @@
             <origin xyz="0 0 0" rpy="0 0 0" />
             <geometry>
-                <box size="0.3 0.02 0.6" />
+                <box size="0.4 0.03 0.8" />
             </geometry>
         </collision>
@@ -296,12 +296,12 @@
     <link name="detector_board2">
         <inertial>
-            <origin xyz="0.0 0.0 -0.28"/>
-            <mass value="2"/>
-            <inertia ixx="0.15" ixy="0.0" ixz="0.0" iyy="0.15" iyz="0.0" izz="0.15"/>
-        </inertial>
-        <visual>
-            <origin xyz="0 0 0" rpy="0 0 0" />
-            <geometry>
-                <box size="0.3 0.02 0.6" />
+            <origin xyz="0.0 0.0 -0.35"/>
+            <mass value="3"/>
+            <inertia ixx="0.2" ixy="0.0" ixz="0.0" iyy="0.2" iyz="0.0" izz="0.2"/>
+        </inertial>
+        <visual>
+            <origin xyz="0 0 0" rpy="0 0 0" />
+            <geometry>
+                <box size="0.4 0.03 0.8" />
             </geometry>
             <material name="detector_blue" />
@@ -310,5 +310,5 @@
             <origin xyz="0 0 0" rpy="0 0 0" />
             <geometry>
-                <box size="0.3 0.02 0.6" />
+                <box size="0.4 0.03 0.8" />
             </geometry>
         </collision>
@@ -318,18 +318,18 @@
         <inertial>
             <origin xyz="0.0 0.0 0.0"/>
-            <mass value="0.25"/>
-            <inertia ixx="0.01" ixy="0.0" ixz="0.0" iyy="0.01" iyz="0.0" izz="0.01"/>
-        </inertial>
-        <visual>
-            <origin xyz="0 0 0" rpy="0 0 0" />
-            <geometry>
-                <box size="0.02 0.02 0.4" />
-            </geometry>
-            <material name="dark_grey" />
-        </visual>
-        <collision>
-            <origin xyz="0 0 0" rpy="0 0 0" />
-            <geometry>
-                <box size="0.02 0.02 0.4" />
+            <mass value="0.35"/>
+            <inertia ixx="0.015" ixy="0.0" ixz="0.0" iyy="0.015" iyz="0.0" izz="0.015"/>
+        </inertial>
+        <visual>
+            <origin xyz="0 0 0" rpy="0 0 0" />
+            <geometry>
+                <box size="0.02 0.02 0.9" />
+            </geometry>
+            <material name="dark_grey" />
+        </visual>
+        <collision>
+            <origin xyz="0 0 0" rpy="0 0 0" />
+            <geometry>
+                <box size="0.02 0.02 0.9" />
             </geometry>
         </collision>
@@ -338,18 +338,18 @@
         <inertial>
             <origin xyz="0.0 0.0 0.0"/>
-            <mass value="0.25"/>
-            <inertia ixx="0.01" ixy="0.0" ixz="0.0" iyy="0.01" iyz="0.0" izz="0.01"/>
-        </inertial>
-        <visual>
-            <origin xyz="0 0 0" rpy="0 0 0" />
-            <geometry>
-                <box size="0.02 0.02 0.4" />
-            </geometry>
-            <material name="dark_grey" />
-        </visual>
-        <collision>
-            <origin xyz="0 0 0" rpy="0 0 0" />
-            <geometry>
-                <box size="0.02 0.02 0.4" />
+            <mass value="0.35"/>
+            <inertia ixx="0.015" ixy="0.0" ixz="0.0" iyy="0.015" iyz="0.0" izz="0.015"/>
+        </inertial>
+        <visual>
+            <origin xyz="0 0 0" rpy="0 0 0" />
+            <geometry>
+                <box size="0.02 0.02 0.9" />
+            </geometry>
+            <material name="dark_grey" />
+        </visual>
+        <collision>
+            <origin xyz="0 0 0" rpy="0 0 0" />
+            <geometry>
+                <box size="0.02 0.02 0.9" />
             </geometry>
         </collision>
@@ -368,5 +368,5 @@
     <!-- Connect board1 to leg1 -->
     <joint name="detector_board1_joint" type="fixed">
-        <origin xyz="0 0 0.4" rpy="0 0 0" />
+        <origin xyz="0 0 0.9" rpy="0 0 0" />
         <parent link="detector_support_leg1"/>
         <child link="detector_board1"/>
@@ -374,5 +374,5 @@
     <!-- Connect board2 to leg2 -->
     <joint name="detector_board2_joint" type="fixed">
-        <origin xyz="0 0 0.4" rpy="0 0 0" />
+        <origin xyz="0 0 0.9" rpy="0 0 0" />
         <parent link="detector_support_leg2"/>
         <child link="detector_board2"/>

File: ranger_mini_v2_gazebo/xacro/ranger_mini_xray_source copy.xacro (robot description, xacro)
@@ -1,24 +1,27 @@
 <?xml version="1.0"?>
-<robot name="ranger_mini_v2"
+<robot name="ranger_mini_xray_source"
     xmlns:xacro="http://ros.org/wiki/xacro">
-    <!-- <xacro:include filename="$(find ranger_mini_v2)/urdf/ranger_l.xacro" />
-    <xacro:include filename="$(find ranger_mini_v2)/urdf/ranger_r.xacro" /> -->
-    <!-- Variables -->
-    <!-- <xacro:property name="M_PI" value="3.14159"/> -->
-    <!-- Vehicle Geometries -->
-    <!-- <xacro:property name="base_x_size" value="1.0" />
-    <xacro:property name="base_y_size" value="0.380000" />
-    <xacro:property name="base_z_size" value="0.210000" />
-    <xacro:property name="wheelbase" value="0.498" />
-    <xacro:property name="track" value="0.58306" />
-    <xacro:property name="wheel_vertical_offset" value="-0.0702" />
-    <xacro:property name="wheel_length" value="1.1653e-01" />
-    <xacro:property name="wheel_radius" value="1.6459e-01" /> -->
+    <!-- Material definitions -->
+    <material name="black">
+        <color rgba="0.1 0.1 0.1 1" />
+    </material>
+    <material name="white">
+        <color rgba="1 1 1 1" />
+    </material>
+    <material name="dark_grey">
+        <color rgba="0.3 0.3 0.3 1" />
+    </material>
+    <material name="metallic_grey">
+        <color rgba="0.7 0.7 0.7 1" />
+    </material>
+    <material name="source_red">
+        <color rgba="0.8 0.2 0.2 1" />
+    </material>
     <!-- Base link -->
     <link name="base_link">
         <inertial>
             <origin xyz="0.0 0.0 0.0"/>
-            <mass value="10"/>
-            <inertia ixx="1" ixy="0.0" ixz="0.0" iyy="1" iyz="0.0" izz="1"/>
+            <mass value="15"/>
+            <inertia ixx="0.5" ixy="0.0" ixz="0.0" iyy="0.5" iyz="0.0" izz="0.5"/>
         </inertial>
         <visual>
@@ -27,4 +30,5 @@
                 <mesh filename="package://ranger_mini_v2/meshes/ranger_base.dae" />
             </geometry>
+            <material name="metallic_grey" />
         </visual>
         <collision>
@@ -46,4 +50,5 @@
                     <mesh filename="package://ranger_mini_v2/meshes/fl.stl" />
             </geometry>
+            <material name="dark_grey" />
         </visual>
         <collision>
@@ -78,4 +83,5 @@
                     <cylinder length="0.01" radius="0.01" />
                 </geometry>
+                <material name="black" />
             </visual>
             <collision>
@@ -108,4 +114,5 @@
                 <mesh filename="package://ranger_mini_v2/meshes/fr.stl" />
             </geometry>
+            <material name="dark_grey" />
         </visual>
         <collision>
@@ -134,4 +141,5 @@
                     <cylinder length="0.01" radius="0.01" />
                 </geometry>
+                <material name="black" />
             </visual>
             <collision>
@@ -164,4 +172,5 @@
                     <mesh filename="package://ranger_mini_v2/meshes/fl.stl" />
             </geometry>
+            <material name="dark_grey" />
         </visual>
         <collision>
@@ -190,4 +199,5 @@
                     <cylinder length="0.01" radius="0.01" />
                 </geometry>
+                <material name="black" />
             </visual>
             <collision>
@@ -220,4 +230,5 @@
                     <mesh filename="package://ranger_mini_v2/meshes/fr.stl" />
             </geometry>
+            <material name="dark_grey" />
         </visual>
         <collision>
@@ -246,4 +257,5 @@
                     <cylinder length="0.01" radius="0.01" />
                 </geometry>
+                <material name="black" />
             </visual>
             <collision>
@@ -345,6 +357,12 @@
       </actuator>
 	</transmission>
+  <!-- Include accessories (3D LiDAR and camera) -->
+  <xacro:include filename="$(find ranger_mini_v2_gazebo)/xacro/accessories_source.urdf.xacro" />
+  <!-- Gazebo ROS Control Plugin -->
   <gazebo>
     <plugin name="gazebo_ros_control" filename="libgazebo_ros_control.so">
+      <robotNamespace>/xray_source</robotNamespace>
+              <robotParam>robot_description</robotParam>
+      <robotSimType>gazebo_ros_control/DefaultRobotHWSim</robotSimType>
     </plugin>
   </gazebo>

File: ranger_mini_v2_gazebo/xacro/ranger_mini_xray_source.xacro (robot description, xacro)
@@ -277,57 +277,29 @@
             <axis xyz="0 1 0" rpy="0 0 0" />
         </joint>
-    <!-- X-ray Source Component -->
-    <link name="xray_source_component">
-        <inertial>
-            <origin xyz="0.0 0.0 0.0"/>
-            <mass value="5"/>
+    <!-- X-ray Source Support Cylinder - Mimics the scanner -->
+    <link name="source_support_cylinder">
+        <inertial>
+            <origin xyz="0.0 0.0 0.6"/>
+            <mass value="8"/>
             <inertia ixx="0.2" ixy="0.0" ixz="0.0" iyy="0.2" iyz="0.0" izz="0.2"/>
         </inertial>
         <visual>
-            <origin xyz="0 0 0" rpy="0 0 0" />
-            <geometry>
-                <cylinder radius="0.1" length="0.3" />
+            <origin xyz="0 0 0.2" rpy="0 0 0" />
+            <geometry>
+                <cylinder radius="0.08" length="1.4"/>
             </geometry>
             <material name="source_red" />
         </visual>
         <collision>
-            <origin xyz="0 0 0" rpy="0 0 0" />
-            <geometry>
-                <cylinder radius="0.1" length="0.3" />
-            </geometry>
-        </collision>
-    </link>
-    <!-- X-ray Source Support -->
-    <link name="xray_source_support">
-        <inertial>
-            <origin xyz="0.0 0.0 0.0"/>
-            <mass value="2"/>
-            <inertia ixx="0.1" ixy="0.0" ixz="0.0" iyy="0.1" iyz="0.0" izz="0.1"/>
-        </inertial>
-        <visual>
-            <origin xyz="0 0 0" rpy="0 0 0" />
-            <geometry>
-                <box size="0.02 0.02 0.4" />
-            </geometry>
-            <material name="dark_grey" />
-        </visual>
-        <collision>
-            <origin xyz="0 0 0" rpy="0 0 0" />
-            <geometry>
-                <box size="0.02 0.02 0.4" />
-            </geometry>
-        </collision>
-    </link>
-    <!-- Connect source support to base -->
-    <joint name="xray_source_support_joint" type="fixed">
-        <origin xyz="0 0 0.2" rpy="0 0 0" />
-        <parent link="base_link"/>
-        <child link="xray_source_support"/>
-    </joint>
-    <!-- Connect source component to support -->
-    <joint name="xray_source_component_joint" type="fixed">
-        <origin xyz="0 0 0.4" rpy="0 0 0" />
-        <parent link="xray_source_support"/>
-        <child link="xray_source_component"/>
+            <origin xyz="0 0 0.2" rpy="0 0 0" />
+            <geometry>
+                <cylinder radius="0.08" length="1.4"/>
+            </geometry>
+        </collision>
+    </link>
+    <joint name="source_support_cylinder_joint" type="fixed">
+        <origin xyz="-0.16 0 0.2" rpy="0 0 0" />
+        <parent link="base_link"/>
+        <child link="source_support_cylinder"/>
     </joint>
 	<transmission name="fl_steering_wheel_trans">

Commit message: change parm

File: ranger_mini_v2_gazebo/xacro/ranger_mini_xray_detector.xacro (robot description, xacro)
@@ -368,5 +368,5 @@
     <!-- Connect board1 to leg1 -->
     <joint name="detector_board1_joint" type="fixed">
-        <origin xyz="0 0 0.9" rpy="0 0 0" />
+        <origin xyz="0 0 0.7" rpy="0 0 0" />
         <parent link="detector_support_leg1"/>
         <child link="detector_board1"/>
@@ -374,5 +374,5 @@
     <!-- Connect board2 to leg2 -->
     <joint name="detector_board2_joint" type="fixed">
-        <origin xyz="0 0 0.9" rpy="0 0 0" />
+        <origin xyz="0 0 0.7" rpy="0 0 0" />
         <parent link="detector_support_leg2"/>
         <child link="detector_board2"/>
