Commit message: add controller

File: ranger_mini_v2_gazebo/xacro/ranger_mini_xray_source.xacro (robot description, xacro)
@@ -287,5 +287,5 @@
             <origin xyz="0 0 0.2" rpy="0 0 0" />
             <geometry>
-                <cylinder radius="0.08" length="1.4"/>
+                <cylinder radius="0.08" length="0.8"/>
             </geometry>
             <material name="source_red" />
@@ -294,5 +294,5 @@
             <origin xyz="0 0 0.2" rpy="0 0 0" />
             <geometry>
-                <cylinder radius="0.08" length="1.4"/>
+                <cylinder radius="0.08" length="0.8"/>
             </geometry>
         </collision>

Commit message: update controller

File: ranger_mini_v2_gazebo/xacro/ranger_mini_xray_source.xacro (robot description, xacro)
@@ -18,13 +18,22 @@
         <color rgba="0.8 0.2 0.2 1" />
     </material>
-    <!-- Base link -->
+    <!-- Base link (aligned with world, no rotation) -->
     <link name="base_link">
         <inertial>
             <origin xyz="0.0 0.0 0.0"/>
-            <mass value="15"/>
+            <mass value="7.5"/>
             <inertia ixx="0.5" ixy="0.0" ixz="0.0" iyy="0.5" iyz="0.0" izz="0.5"/>
         </inertial>
-        <visual>
-            <origin xyz="0 0 0" rpy="1.57 0 3.14 " />
+        <collision>
+            <origin xyz="0 0 -0.1" rpy="0 0 0" />
+            <geometry>
+                <box size="0.5 0.35 0.2"/>
+            </geometry>
+        </collision>
+    </link>
+    <!-- Dummy link for mesh orientation -->
+    <link name="base_mesh">
+        <visual>
+            <origin xyz="0 0 0" rpy="1.57 0 3.14" />
             <geometry>
                 <mesh filename="package://ranger_mini_v2/meshes/ranger_base.dae" />
@@ -32,12 +41,12 @@
             <material name="metallic_grey" />
         </visual>
-        <collision>
-            <origin xyz="0 0 -0.1" rpy="0 0 0" />
-            <geometry>
-                <box size="0.5 0.35 0.2"/>
-            </geometry>
-        </collision>
-    </link>
-   <link name="fl_steering_wheel_link">
+    </link>
+    <joint name="base_mesh_joint" type="fixed">
+        <parent link="base_link"/>
+        <child link="base_mesh"/>
+        <origin xyz="0 0 0" rpy="0 0 0"/>
+    </joint>
+    <!-- Steering and wheel links/joints (all axes and mesh orientations consistent) -->
+    <link name="fl_steering_wheel_link">
         <inertial>
             <origin xyz="0.0 0.0 0.0"/>
@@ -71,37 +80,43 @@
         <axis xyz="0 0 1" rpy="0 0 0" />
         <limit effort="5" velocity="6.28"  lower="-2.1" upper="2.1" />
-    </joint>
-        <link name="fl_wheel_link">
-            <inertial>
-                <mass value="8" />
-                <origin xyz="0 0 0" />
-                <inertia ixx="0.1171" ixy="0" ixz="0" iyy="0.1361" iyz="0" izz="0.1171" />
-            </inertial>
-            <visual>
-                <origin xyz="0 0 0" rpy="1.57 0 0" />
-                <geometry>
-                    <cylinder length="0.01" radius="0.01" />
-                </geometry>
-                <material name="black" />
-            </visual>
-            <collision>
-                <origin xyz="0 0 0" rpy="1.57 0 0" />
-                <geometry>
-                    <cylinder length="0.08" radius="0.08" />
-                </geometry>
-                     <contact>
-                         <ode>
-                        <min_depth>0.001</min_depth>
-                         </ode>
-                    </contact>
-            </collision>
-        </link>
-        <joint name="fl_wheel" type="continuous">
-            <origin xyz="0.03 0.01 -0.12" rpy="0 0 0" />
-            <parent link="fl_steering_wheel_link"/>
-            <child link="fl_wheel_link"/>
-            <axis xyz="0 1 0" rpy="0 0 0" />
-        </joint>
-   <link name="fr_steering_wheel_link">
+        <dynamics damping="0.5" friction="0.1"/>
+    </joint>
+    <link name="fl_wheel_link">
+        <inertial>
+            <mass value="4" />
+            <origin xyz="0 0 0" />
+            <inertia ixx="0.1171" ixy="0" ixz="0" iyy="0.1361" iyz="0" izz="0.1171" />
+        </inertial>
+        <visual>
+            <origin xyz="0 0 0" rpy="1.57 0 0" />
+            <geometry>
+                <cylinder length="0.01" radius="0.01" />
+            </geometry>
+            <material name="black" />
+        </visual>
+        <collision>
+            <origin xyz="0 0 0" rpy="1.57 0 0" />
+            <geometry>
+                <cylinder length="0.08" radius="0.08" />
+            </geometry>
+            <surface>
+                <friction>
+                    <ode>
+                        <mu>0.2</mu>
+                        <mu2>0.1</mu2>
+                    </ode>
+                </friction>
+            </surface>
+        </collision>
+    </link>
+    <joint name="fl_wheel" type="continuous">
+        <origin xyz="0.03 0.01 -0.12" rpy="0 0 0" />
+        <parent link="fl_steering_wheel_link"/>
+        <child link="fl_wheel_link"/>
+        <axis xyz="0 1 0" rpy="0 0 0" />
+        <dynamics damping="0.5" friction="0.1"/>
+    </joint>
+    <!-- Repeat for fr, rl, rr steering and wheel links/joints, all with axis xyz="1 0 0" for wheels and mesh rpy="1.57 0 0" -->
+    <link name="fr_steering_wheel_link">
         <inertial>
             <origin xyz="0.0 0.0 0.0" rpy="0.0 0.0 0.0"/>
@@ -129,37 +144,42 @@
         <axis xyz="0 0 1" rpy="0 0 0" />
         <limit effort="5" velocity="6.28"  lower="-2.1" upper="2.1" />
-    </joint>
-        <link name="fr_wheel_link">
-            <inertial>
-                <mass value="8" />
-                <origin xyz="0 0 0" />
-                <inertia ixx="0.1171" ixy="0" ixz="0" iyy="0.1361" iyz="0" izz="0.1171" />
-            </inertial>
-            <visual>
-                <origin xyz="0 0 0" rpy="1.57 0 0" />
-                <geometry>
-                    <cylinder length="0.01" radius="0.01" />
-                </geometry>
-                <material name="black" />
-            </visual>
-            <collision>
-                <origin xyz="0 0 0" rpy="1.57 0 0" />
-                <geometry>
-                    <cylinder length="0.08" radius="0.085" />
-                </geometry>
-                     <contact>
-                         <ode>
-                        <min_depth>0.001</min_depth>
-                         </ode>
-                    </contact>
-            </collision>
-        </link>
-        <joint name="fr_wheel" type="continuous">
-            <origin xyz="0.0 0.0 -0.12" rpy="0 0 0" />
-            <parent link="fr_steering_wheel_link"/>
-            <child link="fr_wheel_link"/>
-            <axis xyz="0 1 0" rpy="0 0 0" />
-        </joint>
-   <link name="rl_steering_wheel_link">
+        <dynamics damping="0.5" friction="0.1"/>
+    </joint>
+    <link name="fr_wheel_link">
+        <inertial>
+            <mass value="4" />
+            <origin xyz="0 0 0" />
+            <inertia ixx="0.1171" ixy="0" ixz="0" iyy="0.1361" iyz="0" izz="0.1171" />
+        </inertial>
+        <visual>
+            <origin xyz="0 0 0" rpy="1.57 0 0" />
+            <geometry>
+                <cylinder length="0.01" radius="0.01" />
+            </geometry>
+            <material name="black" />
+        </visual>
+        <collision>
+            <origin xyz="0 0 0" rpy="1.57 0 0" />
+            <geometry>
+                <cylinder length="0.08" radius="0.085" />
+            </geometry>
+            <surface>
+                <friction>
+                    <ode>
+                        <mu>0.2</mu>
+                        <mu2>0.1</mu2>
+                    </ode>
+                </friction>
+            </surface>
+        </collision>
+    </link>
+    <joint name="fr_wheel" type="continuous">
+        <origin xyz="0.0 0.0 -0.12" rpy="0 0 0" />
+        <parent link="fr_steering_wheel_link"/>
+        <child link="fr_wheel_link"/>
+        <axis xyz="0 1 0" rpy="0 0 0" />
+        <dynamics damping="0.5" friction="0.1"/>
+    </joint>
+    <link name="rl_steering_wheel_link">
         <inertial>
             <origin xyz="0.0 0.0 0.0" rpy="0.0 0.0 0.0"/>
@@ -187,37 +207,42 @@
         <axis xyz="0 0 1" rpy="0 0 0" />
         <limit effort="5" velocity="6.28"  lower="-2.1" upper="2.1" />
-    </joint>
-        <link name="rl_wheel_link">
-            <inertial>
-                <mass value="8" />
-                <origin xyz="0 0 0" />
-                <inertia ixx="0.1171" ixy="0" ixz="0" iyy="0.1361" iyz="0" izz="0.1171" />
-            </inertial>
-            <visual>
-                <origin xyz="0 0 0" rpy="1.57 0 0" />
-                <geometry>
-                    <cylinder length="0.01" radius="0.01" />
-                </geometry>
-                <material name="black" />
-            </visual>
-            <collision>
-                <origin xyz="0 0 0" rpy="1.57 0 0" />
-                <geometry>
-                    <cylinder length="0.08" radius="0.08" />
-                </geometry>
-                     <contact>
-                         <ode>
-                        <min_depth>0.001</min_depth>
-                         </ode>
-                    </contact>
-            </collision>
-        </link>
-        <joint name="rl_wheel" type="continuous">
-            <origin xyz="0.0 0.0 -0.12 " rpy="0 0 0" />
-            <parent link="rl_steering_wheel_link"/>
-            <child link="rl_wheel_link"/>
-            <axis xyz="0 1 0" rpy="0 0 0" />
-        </joint>
-   <link name="rr_steering_wheel_link">
+        <dynamics damping="0.5" friction="0.1"/>
+    </joint>
+    <link name="rl_wheel_link">
+        <inertial>
+            <mass value="4" />
+            <origin xyz="0 0 0" />
+            <inertia ixx="0.1171" ixy="0" ixz="0" iyy="0.1361" iyz="0" izz="0.1171" />
+        </inertial>
+        <visual>
+            <origin xyz="0 0 0" rpy="1.57 0 0" />
+            <geometry>
+                <cylinder length="0.01" radius="0.01" />
+            </geometry>
+            <material name="black" />
+        </visual>
+        <collision>
+            <origin xyz="0 0 0" rpy="1.57 0 0" />
+            <geometry>
+                <cylinder length="0.08" radius="0.08" />
+            </geometry>
+            <surface>
+                <friction>
+                    <ode>
+                        <mu>0.2</mu>
+                        <mu2>0.1</mu2>
+                    </ode>
+                </friction>
+            </surface>
+        </collision>
+    </link>
+    <joint name="rl_wheel" type="continuous">
+        <origin xyz="0.0 0.0 -0.12 " rpy="0 0 0" />
+        <parent link="rl_steering_wheel_link"/>
+        <child link="rl_wheel_link"/>
+        <axis xyz="0 1 0" rpy="0 0 0" />
+        <dynamics damping="0.5" friction="0.1"/>
+    </joint>
+    <link name="rr_steering_wheel_link">
         <inertial>
             <origin xyz="0.0 0.0 0.0"/>
@@ -245,36 +270,41 @@
         <axis xyz="0 0 1" rpy="0 0 0" />
         <limit effort="5" velocity="6.28"  lower="-2.1" upper="2.1" />
-    </joint>
-        <link name="rr_wheel_link">
-            <inertial>
-                <mass value="8" />
-                <origin xyz="0 0 0" />
-                <inertia ixx="0.1171" ixy="0" ixz="0" iyy="0.1361" iyz="0" izz="0.1171" />
-            </inertial>
-            <visual>
-                <origin xyz="0.0 0.0 0.0" rpy="1.57 0 0" />
-                <geometry>
-                    <cylinder length="0.01" radius="0.01" />
-                </geometry>
-                <material name="black" />
-            </visual>
-            <collision>
-                <origin xyz="0 0 0" rpy="1.57 0 0" />
-                <geometry>
-                    <cylinder length="0.08" radius="0.08" />
-                </geometry>
-                     <contact>
-                         <ode>
-                        <min_depth>0.001</min_depth>
-                         </ode>
-                    </contact>
-            </collision>
-        </link>
-        <joint name="rr_wheel" type="continuous">
-            <origin xyz="0.0 0.0 -0.12 " rpy="0 0 0" />
-            <parent link="rr_steering_wheel_link"/>
-            <child link="rr_wheel_link"/>
-            <axis xyz="0 1 0" rpy="0 0 0" />
-        </joint>
+        <dynamics damping="0.5" friction="0.1"/>
+    </joint>
+    <link name="rr_wheel_link">
+        <inertial>
+            <mass value="4" />
+            <origin xyz="0 0 0" />
+            <inertia ixx="0.1171" ixy="0" ixz="0" iyy="0.1361" iyz="0" izz="0.1171" />
+        </inertial>
+        <visual>
+            <origin xyz="0.0 0.0 0.0" rpy="1.57 0 0" />
+            <geometry>
+                <cylinder length="0.01" radius="0.01" />
+            </geometry>
+            <material name="black" />
+        </visual>
+        <collision>
+            <origin xyz="0 0 0" rpy="1.57 0 0" />
+            <geometry>
+                <cylinder length="0.08" radius="0.08" />
+            </geometry>
+            <surface>
+                <friction>
+                    <ode>
+                        <mu>0.2</mu>
+                        <mu2>0.1</mu2>
+                    </ode>
+                </friction>
+            </surface>
+        </collision>
+    </link>
+    <joint name="rr_wheel" type="continuous">
+        <origin xyz="0.0 0.0 -0.12 " rpy="0 0 0" />
+        <parent link="rr_steering_wheel_link"/>
+        <child link="rr_wheel_link"/>
+        <axis xyz="0 1 0" rpy="0 0 0" />
+        <dynamics damping="0.5" friction="0.1"/>
+    </joint>
     <!-- X-ray Source Support Cylinder - Mimics the scanner -->
     <link name="source_support_cylinder">
